File: Projects/lead/bq24450/bq24450.kicad_pcb (KiCad board)
At the start: 2 copper layers, 11 parts, among them J1 Jack-DC, U1 BQ24450DW

Commit message: new things for charger
Parts:
- added J2: Screw_Terminal_01x02, TerminalBlock:TerminalBlock_bornier-2_P5.08mm, F.Cu at (101.9, 36.5)
- added Q1: PNP, Transistor_Power:MJD127T4GMJD127T4G, F.Cu at (81.7, 90.4)
- C_COMP1: footprint Capacitor_THT:CP_Axial_L29.0mm_D10.0mm_P35.00mm_Horizontal -> Capacitor_THT:C_Disc_D3.0mm_W1.6mm_P2.50mm
- R_A1, R_B1, R_C1, R_D1, R_ISNS1, R_P1, R_T1: footprint Resistor_THT:R_Axial_DIN0309_L9.0mm_D3.2mm_P12.70mm_Horizontal -> Resistor_THT:R_Axial_DIN0207_L6.3mm_D2.5mm_P7.62mm_Horizontal
- U1: footprint Connector_BarrelJack:BarrelJack_Horizontal -> Package_DFN_QFN:BQ24450DW
- moved U1 36.6 mm to (96.5, 78.0)

Commit message: added routing
Parts:
- moved R_D1 45.3 mm to (110.4, 87.0)
- moved R_C1 45.1 mm to (107.0, 87.0), turned to 180 degrees
- moved R_B1 45.0 mm to (109.5, 78.5)
- moved C_COMP1 43.2 mm to (92.5, 79.8), turned to 90 degrees
- moved R_A1 41.6 mm to (109.5, 66.2), turned to -90 degrees
- moved R_P1 33.4 mm to (104.0, 68.0), turned to 180 degrees
- moved Q1 27.8 mm to (88.2, 63.4)
- moved J1 27.4 mm to (86.7, 86.6)
- moved J2 26.4 mm to (118.5, 57.0), turned to -90 degrees
- moved D_EXT1 22.0 mm to (108.8, 59.0), turned to 180 degrees
- moved R_T1 14.6 mm to (84.4, 72.5)
- moved R_ISNS1 13.5 mm to (80.9, 78.5)
- moved U1 4.16 mm to (100.7, 77.9)
Connections:
- net IFB renamed ISNSM
Routing:
- net VFB: track 0.00 -> 37.1 mm
- net ISNSM: track 0.00 -> 23.5 mm
- net Net-(D_EXT1-A): track 0.00 -> 20.2 mm
- net EXT_SUPPLY: track 0.00 -> 18.7 mm
- net PRE_CHG: track 0.00 -> 17.8 mm, vias 0 -> 2
- net Net-(U1-COMP): track 0.00 -> 14.8 mm, vias 0 -> 2
- net STAT1: track 0.00 -> 14.3 mm, vias 0 -> 2
- net PGOOD: track 0.00 -> 8.99 mm
- net CE: track 0.00 -> 8.72 mm
- net Net-(U1-DRVE): track 0.00 -> 7.77 mm
- net SLA_BATTERY: track 0.00 -> 7.46 mm
- net GND: track 0.00 -> 2.57 mm, vias 0 -> 1
- added copper zone on F.Cu, net (none)
- added copper zone on F.Cu, net EXT_SUPPLY
- added copper zone on B.Cu, net GND
- added copper zone on F.Cu, net SLA_BATTERY
Other:
- board outline added: 52 x 55 mm
